File: switch-board/switch_board.kicad_pcb (KiCad board)
At the start: 2 copper layers, 69.8 x 66.3 mm, 38 parts, among them J1 43045-0221, J2 43045-0221, J3 43045-0221, J4 43045-0221, J5 43045-0221, J6 430450421, J7 Conn_01x04_Pin, J8 Conn_01x02_Pin, U1 CSD17578Q5A, U2 CSD17578Q5A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

Commit message: final small mods before ordering
Parts:
- removed MH_1: MountingHole_1, MountingHole:MountingHole_2.2mm_M2_DIN965
- removed REF**: MountingHole_2, MountingHole:MountingHole_2.2mm_M2_DIN965
- removed REF**: MountingHole_3, MountingHole:MountingHole_2.2mm_M2_DIN965
- removed REF**: MountingHole_4, MountingHole:MountingHole_2.2mm_M2_DIN965
- added H3: MountingHole, MountingHole:MountingHole_3.2mm_M3, F.Cu at (123.2, 91.3)
- added H3: MountingHole, MountingHole:MountingHole_3.2mm_M3, F.Cu at (184.9, 91.6)
- added H3: MountingHole, MountingHole:MountingHole_3.2mm_M3, F.Cu at (184.5, 33.5)
- added H3: MountingHole, MountingHole:MountingHole_3.2mm_M3, F.Cu at (122.9, 33.1)
- moved C2 0.55 mm to (173.7, 74.5)
Routing:
- net GND: track 25.1 -> 21.6 mm, vias 24 -> 20
