File: current_sensing/INA228_board/Current_sensing_INA228_board/Current_sensing_INA228_board.kicad_sch (KiCad schematic)
At the start: 25 parts, among them J1 7461096, J2 7461096, J3 Conn_01x06_Pin, U1 INA228

Commit message: Control Board schematics
Parts:
- J1, J2: footprint CONN9_1096_WRE -> footprints:CONN9_1096_WRE
- R1: footprint Resistor_SMD:R_1206_3216Metric -> Resistor_SMD:R_0603_1608Metric
- R10, R2, R3, R4, R5, R6, R7, R8, R9: footprint Resistor_SMD:R_0402_1005Metric -> Resistor_SMD:R_0603_1608Metric
- TP7: value 3.3V -> 5V
Connections:
- net +3.3V renamed +5V
Changed lines of the file:
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@@
 			)
 		)
-		(property "Footprint" "CONN9_1096_WRE"
+		(property "Footprint" "footprints:CONN9_1096_WRE"
 			(at 91.44 133.35 0)
 			(effects
@@
 			)
 		)
-		(property "Value" "+3.3V"
+		(property "Value" "+5V"
 			(at 234.95 108.458 0)
 			(effects
@@
 			)
 		)
-		(property "Footprint" "Resistor_SMD:R_0402_1005Metric"
+		(property "Footprint" "Resistor_SMD:R_0603_1608Metric"
 			(at 226.568 77.47 90)
 			(effects
@@
 			)
 		)
-		(property "Footprint" "Resistor_SMD:R_0402_1005Metric"
+		(property "Footprint" "Resistor_SMD:R_0603_1608Metric"
 			(at 156.972 74.93 90)
 			(effects
@@
 			)
 		)
-		(property "Footprint" "Resistor_SMD:R_0402_1005Metric"
+		(property "Footprint" "Resistor_SMD:R_0603_1608Metric"
 			(at 115.57 95.758 90)
 			(effects
@@
 			)
 		)
-		(property "Footprint" "Resistor_SMD:R_0402_1005Metric"
+		(property "Footprint" "Resistor_SMD:R_0603_1608Metric"
 			(at 203.708 77.47 90)
 			(effects
@@
 			)
 		)
-		(property "Value" "3.3V"
+		(property "Value" "5V"
 			(at 203.2 65.2779 0)
 			(effects
@@
 			)
 		)
-		(property "Footprint" "Resistor_SMD:R_0402_1005Metric"
+		(property "Footprint" "Resistor_SMD:R_0603_1608Metric"
 			(at 176.022 76.2 90)
 			(effects
@@
 			)
 		)
-		(property "Footprint" "Resistor_SMD:R_0402_1005Metric"
+		(property "Footprint" "Resistor_SMD:R_0603_1608Metric"
 			(at 181.61 84.328 90)
 			(effects
@@
 			)
 		)
-		(property "Value" "+3.3V"
-			(at 212.09 60.96 0)
-			(effects
-				(font
-					(size 1.27 1.27)
-				)
+		(property "Value" "+5V"
+			(at 214.63 64.7699 0)
+			(effects
+				(font
+					(size 1.27 1.27)
+				)
+				(justify left)
 			)
 		)
@@
 			)
 		)
-		(property "Footprint" "Resistor_SMD:R_0402_1005Metric"
+		(property "Footprint" "Resistor_SMD:R_0603_1608Metric"
 			(at 213.868 77.47 90)
 			(effects
@@
 			)
 		)
-		(property "Footprint" "CONN9_1096_WRE"
+		(property "Footprint" "footprints:CONN9_1096_WRE"
 			(at 91.44 106.68 0)
 			(effects
@@
 			)
 		)
-		(property "Footprint" "Resistor_SMD:R_0402_1005Metric"
+		(property "Footprint" "Resistor_SMD:R_0603_1608Metric"
 			(at 115.57 103.378 90)
 			(effects
@@
 			)
 		)
-		(property "Footprint" "Resistor_SMD:R_0402_1005Metric"
+		(property "Footprint" "Resistor_SMD:R_0603_1608Metric"
 			(at 162.56 85.598 90)
 			(effects
@@
 			)
 		)
-		(property "Footprint" "Resistor_SMD:R_1206_3216Metric"
+		(property "Footprint" "Resistor_SMD:R_0603_1608Metric"
 			(at 103.632 97.79 90)
 			(effects
