File: control_board/control_board.kicad_sch (KiCad schematic)
At the start: 42 parts, among them J1 Current_sensing, J10 CVM_MUX, J11 CAN connector, J12 CVM_I2C, J13 CVM_MUX, J14 I2C Bus_Connector, J15 Port_B_GPIO, J2 Current_sensing, J3 Shutdown, J4 Shutdown, J5 Shutdown, J6 Current_sensing, J7 Switch_Power, J8 Switch_GPIO, J9 CVM_I2C, SW1 SW_SPST, U1 NUCLEO-L432KC, U10 AZ1117-5.0, U2 TLV76012DBZR, U4 SN65HVD255D, U5 TCA9544A, U6 AP2112K-3.3, U7 DS3502, U8 NHD-1.91-176176UBC3, U9 74LVC1G66

Commit message: Control board PCB finished
Parts:
- removed C1, C2, C4: C, symbol Device:C
- removed C3, C5: 0.1uF, symbol Device:C
- removed D1, D2, D3: LED, symbol Device:LED
- removed J1, J2, J6: Current_sensing, connector1x6:CONN_2125280000_06_MOL, symbol Connector:Conn_01x06_Pin
- removed J10, J13: CVM_MUX, connector1x4:CONN_2125280000_04_MOL, symbol Connector:Conn_01x04_Pin
- removed J11: CAN connector, symbol Connector:Conn_01x02_Pin
- removed J12, J9: CVM_I2C, connector1x4:CONN_2125280000_04_MOL, symbol Connector:Conn_01x04_Pin
- removed J14: I2C Bus_Connector, connector1x12:CONN_2125280000_12_MOL, symbol Connector:Conn_01x12_Pin
- removed J15: Port_B_GPIO, symbol Connector:Conn_01x06_Pin
- removed J3, J4, J5: Shutdown, symbol Connector:Conn_01x02_Pin
- removed J7: Switch_Power, symbol Connector:Conn_01x02_Pin
- removed J8: Switch_GPIO, connector1x4:CONN_2125280000_04_MOL, symbol Connector:Conn_01x04_Pin
- removed R1, R2, R3, R7, R8, R9: R, symbol Device:R
- removed R4: 0, symbol Device:R
- removed R5, R6: 60, symbol Device:R
- removed SW1: SW_SPST, symbol Switch:SW_SPST
- removed U1: NUCLEO-L432KC, NUCLEO-L432KC:MODULE_NUCLEO-L432KC, symbol NUCLEO-L432KC:NUCLEO-L432KC
- removed U10: AZ1117-5.0, symbol Regulator_Linear:AZ1117-5.0
- removed U2: TLV76012DBZR, DBZ0003A_N, symbol 2026-01-24_21-53-39:TLV76012DBZR
- removed U4: SN65HVD255D, Package_SO:SOIC-8_3.9x4.9mm_P1.27mm, symbol Interface_CAN_LIN:SN65HVD255D
- removed U5: TCA9544A, Package_SO:TSSOP-20_4.4x6.5mm_P0.65mm, symbol Interface_Expansion:TCA9544A
- removed U6: AP2112K-3.3, Package_TO_SOT_SMD:SOT-23-5, symbol Regulator_Linear:AP2112K-3.3
- removed U7: DS3502, Package_SO:MSOP-10_3x3mm_P0.5mm, symbol Potentiometer_Digital:DS3502
- removed U8: NHD-1.91-176176UBC3, Connector_PinSocket_2.54mm:PinSocket_2x10_P2.54mm_Vertical, symbol LCD_NHD-1.91-176176UBC3:NHD-1.91-176176UBC3
- removed U9: 74LVC1G66, symbol 74xGxx:74LVC1G66
Connections:
- no-connect marks 3 -> 0
Other:
- added sheet Main_controller (Main_controller.kicad_sch)
- added sheet Memory (Memory.kicad_sch)
- note removed: "2 Mux of the CVM shares the same 4 GPIOs"
- note removed: "Power management"
